File: flextimus-prime.sch (EAGLE design)
At the start: 41 parts, among them T1 2N2222, U1 STM32F042KXU, U2 IP4220CZ6, U3 MCP1802T-3302I/OT

Commit message: better board, for real
Parts:
- removed CN1: (no value), adafruit:USBMOLEX
- removed U2: IP4220CZ6, IP4220CZ6:IP4220CZ6
- added CN2: (no value), adafruit:USBMINIB
Connections:
- removed net USBM: CN1.D+, U2.I/O_4
- removed net USBP: CN1.D-, U2.I/O_1
- net GND: now also CN2.GND; no longer CN1.GND, U2.GND
- net VBUS: now also CN2.VBUS; no longer CN1.VBUS, U2.VP
Other:
- note removed: "Electrostatic Discharge Protection"
- moved on the sheet: C4, C5, C6, C7, C8, D3, FB1, JP5, R8, TP8, U3

Commit message: schematic + board rev 1.2
Parts:
- added C2: 100n, rcl:C-EUC0805
Connections:
- net 3.3V: now also C2.1
- net GND: now also C2.2
Changed lines of the file:
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@@
 <setting verticaltext="up"/>
 </settings>
-<grid distance="0.1" unitdist="inch" unit="inch" style="lines" multiple="1" display="no" altdistance="0.01" altunitdist="inch" altunit="inch"/>
+<grid distance="0.05" unitdist="inch" unit="inch" style="lines" multiple="1" display="yes" altdistance="0.01" altunitdist="inch" altunit="inch"/>
 <layers>
 <layer number="1" name="Top" color="4" fill="1" visible="no" active="no"/>
@@
 <part name="JP3" library="pinhead" library_urn="urn:adsk.eagle:library:325" deviceset="PINHD-1X16" device="" package3d_urn="urn:adsk.eagle:package:22432/2"/>
 <part name="CN2" library="adafruit" library_urn="urn:adsk.eagle:library:420" deviceset="USB" device="MINIB"/>
+<part name="C2" library="rcl" library_urn="urn:adsk.eagle:library:334" deviceset="C-EU" device="C0805" package3d_urn="urn:adsk.eagle:package:23617/2" value="100n"/>
+<part name="GND15" library="SparkFun-PowerSymbols" library_urn="urn:adsk.eagle:library:530" deviceset="GND" device=""/>
 </parts>
 <sheets>
@@
 <text x="-116.84" y="80.01" size="1.778" layer="97">Derivative schematic based off of http://ebrombaugh.studionebula.com/embedded/stm32f042breakout/stm32f042f_breakout_schematic.pdf</text>
 <wire x1="-135.89" y1="-68.58" x2="-135.89" y2="-116.84" width="0.1524" layer="94"/>
-<wire x1="-135.89" y1="-116.84" x2="27.94" y2="-116.84" width="0.1524" layer="94"/>
-<wire x1="27.94" y1="-116.84" x2="27.94" y2="-68.58" width="0.1524" layer="94"/>
-<wire x1="27.94" y1="-68.58" x2="-135.89" y2="-68.58" width="0.1524" layer="94"/>
+<wire x1="-135.89" y1="-116.84" x2="30.48" y2="-116.84" width="0.1524" layer="94"/>
+<wire x1="30.48" y1="-116.84" x2="30.48" y2="-68.58" width="0.1524" layer="94"/>
+<wire x1="30.48" y1="-68.58" x2="-135.89" y2="-68.58" width="0.1524" layer="94"/>
 <text x="-133.35" y="-72.39" size="1.778" layer="94">Power</text>
 <wire x1="60.96" y1="-16.51" x2="125.73" y2="-16.51" width="0.1524" layer="94"/>
@@
 <wire x1="-116.84" y1="-25.4" x2="-116.84" y2="33.02" width="0.1524" layer="94"/>
 <text x="-78.74" y="31.75" size="1.778" layer="94" rot="R180">User Interface 2 (LCD Screen)</text>
-<wire x1="-60.96" y1="-58.42" x2="-60.96" y2="35.56" width="0.1524" layer="94"/>
+<wire x1="-60.96" y1="-66.04" x2="-60.96" y2="35.56" width="0.1524" layer="94"/>
 <wire x1="-60.96" y1="35.56" x2="43.18" y2="35.56" width="0.1524" layer="94"/>
-<wire x1="43.18" y1="35.56" x2="43.18" y2="-58.42" width="0.1524" layer="94"/>
-<wire x1="43.18" y1="-58.42" x2="-60.96" y2="-58.42" width="0.1524" layer="94"/>
+<wire x1="43.18" y1="35.56" x2="43.18" y2="-66.04" width="0.1524" layer="94"/>
+<wire x1="43.18" y1="-66.04" x2="-60.96" y2="-66.04" width="0.1524" layer="94"/>
 <text x="-39.37" y="34.29" size="1.778" layer="94" rot="R180">Microprocessor</text>
 <text x="88.9" y="-151.13" size="1.778" layer="97">Team 7:
@@
 <instance part="GND20" gate="1" x="113.03" y="-58.42"/>
 <instance part="GND4" gate="1" x="69.85" y="-40.64"/>
-<instance part="SUPPLY4" gate="G$1" x="-8.89" y="-48.26"/>
+<instance part="SUPPLY4" gate="G$1" x="-7.62" y="-48.26"/>
 <instance part="JP3" gate="A" x="-88.9" y="5.08"/>
 <instance part="CN2" gate="G$1" x="-121.92" y="-91.44"/>
+<instance part="C2" gate="G$1" x="-5.08" y="-53.34"/>
+<instance part="GND15" gate="1" x="-5.08" y="-63.5"/>
 </instances>
 <busses>
@@
 </segment>
 <segment>
-<pinref part="U1" gate="B" pin="VDDIO2"/>
-<pinref part="SUPPLY4" gate="G$1" pin="3.3V"/>
-</segment>
-<segment>
 <wire x1="-91.44" y1="20.32" x2="-99.06" y2="20.32" width="0.1524" layer="91"/>
 <wire x1="-99.06" y1="20.32" x2="-99.06" y2="17.78" width="0.1524" layer="91"/>
@@
 <pinref part="JP3" gate="A" pin="2"/>
 <pinref part="JP3" gate="A" pin="3"/>
+</segment>
+<segment>
+<pinref part="U1" gate="B" pin="VDDIO2"/>
+<wire x1="-8.89" y1="-48.26" x2="-7.62" y2="-48.26" width="0.1524" layer="91"/>
+<pinref part="C2" gate="G$1" pin="1"/>
+<wire x1="-7.62" y1="-48.26" x2="-5.08" y2="-48.26" width="0.1524" layer="91"/>
+<wire x1="-5.08" y1="-50.8" x2="-5.08" y2="-48.26" width="0.1524" layer="91"/>
+<pinref part="SUPPLY4" gate="G$1" pin="3.3V"/>
+<junction x="-7.62" y="-48.26"/>
 </segment>
 </net>
@@
 <pinref part="JP3" gate="A" pin="1"/>
 </segment>
+<segment>
+<pinref part="C2" gate="G$1" pin="2"/>
+<pinref part="GND15" gate="1" pin="GND"/>
+<wire x1="-5.08" y1="-60.96" x2="-5.08" y2="-58.42" width="0.1524" layer="91"/>
+</segment>
 </net>
 <net name="SWDIO" class="0">
@@
 <pinref part="C7" gate="G$1" pin="1"/>
 <wire x1="7.62" y1="-86.36" x2="7.62" y2="-88.9" width="0.1524" layer="91"/>
-<wire x1="7.62" y1="-86.36" x2="16.51" y2="-86.36" width="0.1524" layer="91"/>
+<wire x1="7.62" y1="-86.36" x2="15.24" y2="-86.36" width="0.1524" layer="91"/>
 <junction x="7.62" y="-86.36"/>
 <pinref part="C8" gate="G$1" pin="1"/>
+<wire x1="15.24" y1="-86.36" x2="16.51" y2="-86.36" width="0.1524" layer="91"/>
 <wire x1="16.51" y1="-86.36" x2="16.51" y2="-88.9" width="0.1524" layer="91"/>
-<wire x1="16.51" y1="-86.36" x2="21.59" y2="-86.36" width="0.1524" layer="91"/>
-<junction x="16.51" y="-86.36"/>
-<label x="19.05" y="-86.36" size="1.778" layer="95"/>
 <pinref part="FB1" gate="G$1" pin="2"/>
 <wire x1="2.54" y1="-86.36" x2="7.62" y2="-86.36" width="0.1524" layer="91"/>
+<wire x1="16.51" y1="-86.36" x2="20.32" y2="-86.36" width="0.1524" layer="91"/>
+<label x="20.32" y="-86.36" size="1.778" layer="95" xref="yes"/>
+<junction x="16.51" y="-86.36"/>
 </segment>
 </net>
